File: 750-THR-Earthtyper/750-THR-Earthtyper.kicad_pcb (KiCad board)
At the start: 2 copper layers, 165 parts, among them K1 KEYSW, K10 KEYSW, K11 KEYSW, K12 KEYSW, K13 KEYSW, K14 KEYSW, K15 KEYSW, K16 KEYSW, K17 KEYSW, K18 KEYSW, K19 KEYSW, K2 KEYSW, K20 KEYSW, K21 KEYSW, K22 KEYSW, K23 KEYSW, K24 KEYSW, K25 KEYSW, K26 KEYSW, K27 KEYSW, K28 KEYSW, K29 KEYSW, K3 KEYSW, K30 KEYSW, K31 KEYSW, K32 KEYSW, K33 KEYSW, K34 KEYSW, K35 KEYSW, K36 KEYSW, K37 KEYSW, K38 KEYSW, K39 KEYSW, K4 KEYSW, K40 KEYSW, K41 KEYSW, K42 KEYSW, K43 KEYSW, K44 KEYSW, K45 KEYSW, K46 KEYSW, K47 KEYSW, K48 KEYSW, K49 KEYSW, K5 KEYSW, K50 KEYSW, K51 KEYSW, K52 KEYSW, K53 KEYSW, K54 KEYSW, K55 KEYSW, K56 KEYSW, K57 KEYSW, K58 KEYSW, K59 KEYSW, K6 KEYSW, K60 KEYSW, K61 KEYSW, K62 KEYSW, K63 KEYSW, K64 KEYSW, K65 KEYSW, K66 KEYSW, K67 KEYSW, K68 KEYSW, K69 KEYSW, K7 KEYSW, K70 KEYSW, K71 KEYSW, K72 KEYSW, K73 KEYSW, K74 KEYSW, K75 KEYSW, K76 KEYSW, K77 KEYSW, K78 KEYSW, K79 KEYSW, K8 KEYSW, K80 KEYSW, K81 KEYSW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

Commit message: added alot of things
Parts:
- added G***: LOGO, LOGO, F.Cu at (145.8, -74.2)
- D1, D10, D11, D12, D13, D14, D15, D16, D17, D18, D19, D2, D20, D21, D22, D23, D24, D25, D26, D27, D28, D29, D3, D30, D31, D32, D33, D34, D35, D36, D37, D38, D39, D4, D40, D41, D42, D43, D44, D45, D46, D47, D48, D49, D5, D50, D51, D52, D53, D54, D55, D56, D57, D58, D59, D6, D60, D61, D62, D63, D64, D65, D66, D67, D68, D69, D7, D70, D71, D72, D73, D74, D75, D76, D77, D78, D79, D8, D80, D81, D82, D9: footprint keyboard_parts.pretty-master:D_SOD123 -> keyboard_parts.pretty-master:D_SOD123_axial
- K1, K10, K11, K12, K13, K14, K15, K16, K17, K18, K19, K2, K20, K21, K22, K23, K24, K25, K26, K27, K28, K29, K3, K30, K31, K32, K33, K34, K35, K36, K37, K38, K39, K4, K40, K41, K42, K43, K44, K45, K46, K47, K48, K49, K5, K50, K51, K52, K53, K54, K55, K56, K57, K58, K59, K6, K60, K61, K62, K63, K64, K65, K66, K67, K68, K69, K7, K70, K71, K72, K73, K74, K75, K76, K77, K78, K79, K8, K80, K81, K82, K9: moved to F.Cu
- moved D82 365.1 mm to (286.3, -14.2)
- moved D59 360.9 mm to (286.3, -56.8)
- moved D15 360.3 mm to (286.3, -118.4)
- moved D45 359.9 mm to (286.3, -75.8)
- moved D30 358.7 mm to (286.3, -94.7)
- moved D14 357.2 mm to (262.6, -118.4)
- moved D80 350.1 mm to (267.3, -33.2)
- moved D81 345.9 mm to (267.3, -14.2)
- moved D13 335.8 mm to (238.9, -118.4)
- moved D44 332.0 mm to (257.8, -75.8)
- moved D29 326.8 mm to (253.1, -94.7)
- moved D58 325.9 mm to (250.7, -56.8)
- moved D79 325.7 mm to (248.4, -14.2)
- moved D12 318.5 mm to (219.9, -118.4)
- moved D28 318.4 mm to (224.7, -94.7)
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Routing:
- net Net-(U1-PF6): track 0.00 -> 391.7 mm
- net Net-(D1-K): track 0.00 -> 386.8 mm, vias 0 -> 14
- net Net-(D16-K): track 0.00 -> 356.1 mm, vias 0 -> 18
- net Net-(D31-K): track 0.00 -> 345.4 mm, vias 0 -> 23
- net Net-(D72-K): track 0.00 -> 344.3 mm
- net Net-(D46-K): track 0.00 -> 324.5 mm, vias 0 -> 27
- net Net-(U1-PF5): track 0.00 -> 298.8 mm, vias 0 -> 2
- net Net-(U1-PF4): track 0.00 -> 285.4 mm, vias 0 -> 2
- net Net-(D60-K): track 0.00 -> 272.0 mm, vias 0 -> 10
- net Net-(U1-PF1): track 0.00 -> 255.3 mm, vias 0 -> 4
- net Net-(U1-PF0): track 0.00 -> 230.6 mm, vias 0 -> 2
- net Net-(U1-PE6): track 0.00 -> 218.1 mm
- net Net-(U1-PB7): track 0.00 -> 207.1 mm, vias 0 -> 2
- net Net-(U1-PD7): track 0.00 -> 199.8 mm, vias 0 -> 3
- net Net-(U1-PD5): track 0.00 -> 190.4 mm, vias 0 -> 1
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Other:
- board outline added: 307.9 x 123.2 mm

Commit message: fixed an error with the schematic and organized the schematic
Parts:
- K71: footprint keebs.pretty-master:Mx_Alps_175 -> keebs.pretty-master:Mx_Alps_100
- K72, K73, K74: footprint keebs.pretty-master:Mx_Alps_125 -> keebs.pretty-master:Mx_Alps_100
- K75: footprint keebs.pretty-master:Mx_Alps_625 -> keebs.pretty-master:Mx_Alps_100
Connections:
- net Net-(D1-K) renamed row0
- net Net-(D16-K) renamed row1
- net Net-(D31-K) renamed row2
- net Net-(D46-K) renamed row3
- net Net-(D60-K) renamed row4
- net Net-(D72-K) renamed row5
- net Net-(U1-PB7) renamed col0
- net Net-(U1-PC6) renamed col1
- net Net-(U1-PC7) renamed col2
- net Net-(U1-PD0) renamed col3
- net Net-(U1-PD1) renamed col4
- net Net-(U1-PD2) renamed col5
- net Net-(U1-PD3) renamed col6
- net Net-(U1-PD4) renamed col7
- net Net-(U1-PD5) renamed col8
- net Net-(U1-PD7) renamed col9
- net Net-(U1-PE6) renamed col10
- net Net-(U1-PF0) renamed col11
- net Net-(U1-PF1) renamed col12
- net Net-(U1-PF4) renamed col13
- net Net-(U1-PF5) renamed col14
- net Net-(U1-PF6) renamed col15
