File: 750-THR-Earthtyper/750-THR-Earthtyper.kicad_sch (KiCad schematic)
At the start: 165 parts, among them K1 KEYSW, K10 KEYSW, K11 KEYSW, K12 KEYSW, K13 KEYSW, K14 KEYSW, K15 KEYSW, K16 KEYSW, K17 KEYSW, K18 KEYSW, K19 KEYSW, K2 KEYSW, K20 KEYSW, K21 KEYSW, K22 KEYSW, K23 KEYSW, K24 KEYSW, K25 KEYSW, K26 KEYSW, K27 KEYSW, K28 KEYSW, K29 KEYSW, K3 KEYSW, K30 KEYSW, K31 KEYSW, K32 KEYSW, K33 KEYSW, K34 KEYSW, K35 KEYSW, K36 KEYSW, K37 KEYSW, K38 KEYSW, K39 KEYSW, K4 KEYSW, K40 KEYSW, K41 KEYSW, K42 KEYSW, K43 KEYSW, K44 KEYSW, K45 KEYSW, K46 KEYSW, K47 KEYSW, K48 KEYSW, K49 KEYSW, K5 KEYSW, K50 KEYSW, K51 KEYSW, K52 KEYSW, K53 KEYSW, K54 KEYSW, K55 KEYSW, K56 KEYSW, K57 KEYSW, K58 KEYSW, K59 KEYSW, K6 KEYSW, K60 KEYSW, K61 KEYSW, K62 KEYSW, K63 KEYSW, K64 KEYSW, K65 KEYSW, K66 KEYSW, K67 KEYSW, K68 KEYSW, K69 KEYSW, K7 KEYSW, K70 KEYSW, K71 KEYSW, K72 KEYSW, K73 KEYSW, K74 KEYSW, K75 KEYSW, K76 KEYSW, K77 KEYSW, K78 KEYSW, K79 KEYSW, K8 KEYSW, K80 KEYSW, K81 KEYSW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

Commit message: added alot of things
Parts:
- D1, D10, D11, D12, D13, D14, D15, D16, D17, D18, D19, D2, D20, D21, D22, D23, D24, D25, D26, D27, D28, D29, D3, D30, D31, D32, D33, D34, D35, D36, D37, D38, D39, D4, D40, D41, D42, D43, D44, D45, D46, D47, D48, D49, D5, D50, D51, D52, D53, D54, D55, D56, D57, D58, D59, D6, D60, D61, D62, D63, D64, D65, D66, D67, D68, D69, D7, D70, D71, D72, D73, D74, D75, D76, D77, D78, D79, D8, D80, D81, D82, D9: footprint keyboard_parts.pretty-master:D_SOD123 -> keyboard_parts.pretty-master:D_SOD123_axial

Commit message: updated the pcb to use net labels (thank you kai)
Connections:
- net row1: now reaches D16.1 (K), D17.1 (K), D18.1 (K), D19.1 (K), D20.1 (K), D21.1 (K), D22.1 (K), D23.1 (K), D24.1 (K), D25.1 (K), D26.1 (K), D27.1 (K), D28.1 (K), D29.1 (K), D30.1 (K), U1.4 (PB2)
- net col12: now reaches K12.2, K28.2, K42.2, K57.2, K78.2, U1.27 (PF1)
- net col10: now reaches K10.2, K26.2, K40.2, K55.2, K69.2, K76.2, U1.31 (PE6)
- net col3: now reaches K19.2, K33.2, K4.2, K48.2, K62.2, K74.2, U1.7 (PD0)
- net row4: now reaches D60.1 (K), D61.1 (K), D62.1 (K), D63.1 (K), D64.1 (K), D65.1 (K), D66.1 (K), D67.1 (K), D68.1 (K), D69.1 (K), D70.1 (K), D71.1 (K), D80.1 (K), U1.21 (PB5)
- net row3: now reaches D46.1 (K), D47.1 (K), D48.1 (K), D49.1 (K), D50.1 (K), D51.1 (K), D52.1 (K), D53.1 (K), D54.1 (K), D55.1 (K), D56.1 (K), D57.1 (K), D58.1 (K), D59.1 (K), U1.20 (PB4)
- net row5: now reaches D72.1 (K), D73.1 (K), D74.1 (K), D75.1 (K), D76.1 (K), D77.1 (K), D78.1 (K), D79.1 (K), D81.1 (K), D82.1 (K), U1.22 (PB6)
- net row2: now reaches D31.1 (K), D32.1 (K), D33.1 (K), D34.1 (K), D35.1 (K), D36.1 (K), D37.1 (K), D38.1 (K), D39.1 (K), D40.1 (K), D41.1 (K), D42.1 (K), D43.1 (K), D44.1 (K), D45.1 (K), U1.5 (PB3)
- net col4: now reaches K20.2, K34.2, K49.2, K5.2, K63.2, U1.8 (PD1)
- net row0: now reaches D1.1 (K), D10.1 (K), D11.1 (K), D12.1 (K), D13.1 (K), D14.1 (K), D15.1 (K), D2.1 (K), D3.1 (K), D4.1 (K), D5.1 (K), D6.1 (K), D7.1 (K), D8.1 (K), D9.1 (K), U1.2 (PB0)
- net col13: now reaches K13.2, K43.2, K58.2, K71.2, K79.2, U1.26 (PF4)
- net col8: now reaches K24.2, K38.2, K53.2, K67.2, K8.2, U1.13 (PD5)
- net col14: now reaches K14.2, K29.2, K44.2, K80.2, K81.2, U1.25 (PF5)
- net col2: now reaches K18.2, K3.2, K32.2, K47.2, K61.2, U1.12 (PC7)
- net col15: now reaches K15.2, K30.2, K45.2, K59.2, K82.2, U1.24 (PF6)
- net col6: now reaches K22.2, K36.2, K51.2, K6.2, K65.2, K75.2, U1.10 (PD3)
- net at K21.2, K35.2, K50.2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: no longer U1.9 (PD2)
- net col0: now reaches K1.2, K16.2, K31.2, K46.2, K60.2, K72.2, U1.6 (PB7)
- net col1: now reaches K17.2, K2.2, K73.2, U1.11 (PC6)
- net col9: now reaches K25.2, K39.2, K54.2, K68.2, K9.2, U1.19 (PD7)
- net col11: now reaches K11.2, K27.2, K41.2, K56.2, K70.2, K77.2, U1.28 (PF0)
- net col7: now reaches K23.2, K37.2, K52.2, K66.2, K7.2, U1.17 (PD4)
- new net col5: U1.9 (PD2)

Commit message: fixed an error with the schematic and organized the schematic
Parts:
- K71: footprint keebs.pretty-master:Mx_Alps_175 -> keebs.pretty-master:Mx_Alps_100
- K72, K73, K74: footprint keebs.pretty-master:Mx_Alps_125 -> keebs.pretty-master:Mx_Alps_100
- K75: footprint keebs.pretty-master:Mx_Alps_625 -> keebs.pretty-master:Mx_Alps_100
Connections:
- net col5: now also K21.2, K35.2, K50.2, K64.2
- no-connect marks 12 -> 10
Other:
- moved on the sheet: D10, D11, D12, D14, D15, D18, D19, D2, D20, D21, D22, D23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
